File: g6uw_relay.kicad_pcb (KiCad board)
At the start: 2 copper layers, 80 x 100 mm, 27 parts, among them J1 Barrel_Jack_Switch, J2 083-1R, J3 083-1R, J4 083-1R, Q1 IRF8721PBF-1, U1 MCP1804x-3002xDB, U2 ORJ-5

Commit message: Version sent to JLCPCB
Parts:
- added J5: Conn_01x02_Male, Connector_PinSocket_2.54mm:PinSocket_1x02_P2.54mm_Vertical, F.Cu at (112.5, 123.8)
- added M1: Logo_10mmx10mm, Misc_WUT:Logo_10mmx10mm_Monocle, F.Cu at (102.5, 90.0)
- moved J2 0.50 mm to (165.5, 65.0)
- moved J3 0.50 mm to (165.5, 135.0)
- moved J4 0.50 mm to (165.5, 100.0)
Routing:
- net +3V3: track 21.8 -> 27.7 mm
- net Net-(C5-Pad1): track 24.0 -> 29.9 mm
Other:
- outline, holes or cut-outs redrawn
- board text added: "MØWUT"
- board text added: "Short to test"
