File: Panels/back_panel/back/back.kicad_pcb (KiCad board)
At the start: 2 copper layers, 108.5 x 44.5 mm, 4 parts

Commit message: Version sent to JLCPCB
Other:
- board text added: "Auto-TOS3R"
Changed lines of the file:
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@@
   (general
     (thickness 1.6)
-    (drawings 40)
+    (drawings 41)
     (tracks 159)
     (zones 0)
@@
     (35 F.Paste user)
     (36 B.SilkS user)
-    (37 F.SilkS user hide)
+    (37 F.SilkS user)
     (38 B.Mask user)
     (39 F.Mask user)
@@
     (aux_axis_origin 0 0)
     (grid_origin 150 99.5)
-    (visible_elements FFFFFF7F)
+    (visible_elements 7FFFFFFF)
     (pcbplotparams
       (layerselection 0x010fc_ffffffff)
@@
       (outputformat 1)
       (mirror false)
-      (drillshape 1)
+      (drillshape 0)
       (scaleselection 1)
       (outputdirectory ""))
@@
       (net 1 GND))
   )
+  (gr_text Auto-TOS3R (at 150 117) (layer F.SilkS)
+    (effects (font (size 1.5 1.5) (thickness 0.3)))
+  )
   (gr_line (start 204.25 80.25) (end 204.25 118.75) (layer Edge.Cuts) (width 0.05))
